File: badge/badge-18650/badge-18650.kicad_pcb (KiCad board)
At the start: 2 copper layers, 179.1 x 63.5 mm, 65 parts, among them J1 Conn_01x03, J2 io_connector, J4 io_connector, J5 USB_C_Receptacle_USB2.0, Q1 BSS138, Q2 BSS138, Q3 BSS138, Q4 BSS138, SW1 SW_DIP_x04, U1 NS8002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

Commit message: badge add on, as submitted.
Other:
- board text added: "JLCJLCJLCJLC"
Changed lines of the file:
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@@
       (viasonmask false)
       (mode 1)
-      (useauxorigin true)
+      (useauxorigin false)
       (hpglpennumber 1)
       (hpglpenspeed 20)
@@
     (effects (font (size 3 3) (thickness 0.5)) (justify mirror))
   )
+  (gr_text "JLCJLCJLCJLC" (at 147.32 110.1852) (layer "B.SilkS")
+    (effects (font (size 2 2) (thickness 0.3)) (justify mirror))
+  )
   (gr_text "@TomKeddie\nSupercon 2022" (at 123.952 133.604) (layer "B.SilkS")
