File: badge/badge-18650/badge-18650.kicad_sch (KiCad schematic)
At the start: 62 parts, among them J1 Conn_01x03, J2 io_connector, J4 io_connector, J5 USB_C_Receptacle_USB2.0, Q1 BSS138, Q2 BSS138, Q3 BSS138, Q4 BSS138, SW1 SW_DIP_x04, U1 NS8002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

Commit message: badge add on, as submitted.
Parts:
- U4: LCSC (none) -> C62244
Changed lines of the file:
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@@
+      (effects (font (size 1.27 1.27)) hide)
+    )
+    (property "LCSC" "C62244" (id 4) (at 132.08 176.53 0)
       (effects (font (size 1.27 1.27)) hide)
     )
